File: samples/files/summe_v6/main.kicad_sch (KiCad schematic)
At the start: 6 parts, among them U1 TL072

Commit message: schema refactoring
Other:
- company: (none) -> Company
Changed lines of the file:
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@@
     (date "2021-05-30")
     (rev "R02")
+    (company "Company")
     (comment 1 "schema for pcb")
     (comment 2 "DC coupled mixer")
+    (comment 3 "comment 3")
     (comment 4 "License CC BY 4.0 - Attribution 4.0 International")
+    (comment 5 "comment 5")
+    (comment 6 "comment 6")
+    (comment 7 "comment 7")
+    (comment 8 "comment 8")
+    (comment 9 "comment 9")
   )
   (junction (at 93.98 148.59) (diameter 0) (color 0 0 0 0)
@@
     (pin "2")
     (pin "3")
-  )
-  (symbol (lib_id "Device:C") (at 93.98 160.02 0)
+    (pin "5")
+    (pin "6")
+    (pin "7")
+    (pin "4")
+    (pin "8")
+  )
+  (symbol (lib_id "Device:C") (at 93.98 160.02 0) (unit 1)
     (in_bom yes) (on_board yes)
     (property "Reference" "C2" (id 0) (at 96.901 158.8516 0)
@@
     (pin "2")
   )
-  (symbol (lib_id "Device:C") (at 93.98 152.4 0)
+  (symbol (lib_id "Device:C") (at 93.98 152.4 0) (unit 1)
     (in_bom yes) (on_board yes)
     (property "Reference" "C1" (id 0) (at 96.901 151.2316 0)
@@
     (pin "2")
   )
-  (symbol (lib_id "power:+15V") (at 93.98 148.59 0)
+  (symbol (lib_id "power:+15V") (at 93.98 148.59 0) (unit 1)
     (in_bom yes) (on_board yes)
     (property "Reference" "#PWR07" (id 0) (at 93.98 152.4 0)
@@
     (pin "1")
   )
-  (symbol (lib_id "power:-15V") (at 93.98 163.83 180)
+  (symbol (lib_id "power:-15V") (at 93.98 163.83 180) (unit 1)
     (in_bom yes) (on_board yes)
     (property "Reference" "#PWR08" (id 0) (at 93.98 166.37 0)
@@
     (pin "1")
   )
-  (symbol (lib_id "power:GND") (at 87.63 158.75 0)
+  (symbol (lib_id "power:GND") (at 87.63 158.75 0) (unit 1)
     (in_bom yes) (on_board yes)
     (property "Reference" "#PWR06" (id 0) (at 87.63 165.1 0)
@@
       (effects (font (size 1.27 1.27)) hide)
     )
+    (pin "1")
+    (pin "2")
+    (pin "3")
+    (pin "5")
+    (pin "6")
+    (pin "7")
     (pin "4")
     (pin "8")
@@
       (effects (font (size 1.27 1.27)) hide)
     )
+    (pin "1")
+    (pin "2")
+    (pin "3")
     (pin "5")
     (pin "6")
     (pin "7")
+    (pin "4")
+    (pin "8")
   )
   (sheet_instances
